Commit message: day::2 almost got robot_description

File: chefbot_description/robots/chefbot_circles_kinect.urdf.xacro (robot description, xacro)
@@ -6,6 +6,5 @@
 -->
 <robot name="turtlebot" xmlns:xacro="http://ros.org/wiki/xacro">
-<!--  <xacro:include filename="$(find turtlebot_description)/urdf/turtlebot_library.urdf.xacro" /> -->
-  <xacro:include filename="$(find black_dount_description)/urdf/black_dount_rviz_library.urdf.xacro" />
+  <xacro:include filename="$(find chefbot_description)/urdf/chefbot_library.urdf.xacro" />
   <kobuki/>
   <stack_hexagons parent="base_link"/>

File: chefbot_description/urdf/bkup/chefbot_base.urdf.xacro (robot description, xacro)
@@ -7,6 +7,6 @@
  -->
 <robot name="kobuki" xmlns:xacro="http://ros.org/wiki/xacro">
-  <xacro:include filename="$(find black_dount_description)/urdf/common_properties.urdf.xacro"/>
-  <xacro:include filename="$(find black_dount_description)/urdf/black_dount_base_gazebo.urdf.xacro"/>
+  <xacro:include filename="$(find chefbot_description)/urdf/common_properties.urdf.xacro"/>
+  <xacro:include filename="$(find chefbot_description)/urdf/chefbot_base_gazebo.urdf.xacro"/>
   <!-- Kobuki -->
   <xacro:macro name="kobuki">
@@ -30,5 +30,5 @@
         <geometry>
           <!-- new mesh -->
-          <mesh filename="package://black_dount_description/meshes/base_plate.dae" />
+          <mesh filename="package://chefbot_description/meshes/base_plate.dae" />
         </geometry>
 <!--        <origin xyz="0.001 0 0.05199" rpy="0 0 ${M_PI/2}"/> -->
@@ -66,5 +66,5 @@
       <visual>
         <geometry>
-          <mesh filename="package://black_dount_description/meshes/wheel.dae"/>
+          <mesh filename="package://chefbot_description/meshes/wheel.dae"/>
         </geometry>
         <origin xyz="0 0 0" rpy="0 0 0"/>
@@ -93,5 +93,5 @@
       <visual>
         <geometry>
-          <mesh filename="package://black_dount_description/meshes/wheel.dae"/>
+          <mesh filename="package://chefbot_description/meshes/wheel.dae"/>
         </geometry>
         <origin xyz="0 0 0" rpy="0 0 0"/>

File: chefbot_description/urdf/bkup/chefbot_base_gazebo.urdf.xacro (robot description, xacro)
@@ -1,6 +1,6 @@
 <?xml version="1.0"?>
-<robot name="black_donut" xmlns:xacro="http://ros.org/wiki/xacro">
-  <xacro:macro name="black_donut">
-	  <gazebo reference="black_dount_wheel_left_link">
+<robot name="kobuki_sim" xmlns:xacro="http://ros.org/wiki/xacro">
+  <xacro:macro name="kobuki_sim">
+	  <gazebo reference="wheel_left_link">
 	    <mu1>1.0</mu1>
 	    <mu2>1.0</mu2>
@@ -10,5 +10,5 @@
 	    <maxVel>1.0</maxVel>
 	  </gazebo>
-	  <gazebo reference="black_dount_wheel_right_link">
+	  <gazebo reference="wheel_right_link">
 	    <mu1>1.0</mu1>
 	    <mu2>1.0</mu2>
@@ -18,5 +18,5 @@
 	    <maxVel>1.0</maxVel>
 	  </gazebo>
-	  <gazebo reference="black_dount_caster_front_link">
+	  <gazebo reference="caster_front_link">
 	    <mu1>0.0</mu1>
 	    <mu2>0.0</mu2>
@@ -26,5 +26,5 @@
 	    <maxVel>1.0</maxVel>
 	  </gazebo>
-	  <gazebo reference="black_dount_caster_back_link">
+	  <gazebo reference="caster_back_link">
 	    <mu1>0.0</mu1>
 	    <mu2>0.0</mu2>

File: chefbot_description/urdf/chefbot_base.urdf.xacro (robot description, xacro)
@@ -6,10 +6,10 @@
       kobuki_description/launch/view_model.launch
  -->
-<robot name="black_dount" xmlns:xacro="http://ros.org/wiki/xacro">
-  <xacro:include filename="$(find black_dount_description)/urdf/common_properties.urdf.xacro"/>
-  <xacro:include filename="$(find black_dount_description)/urdf/black_dount_base_gazebo.urdf.xacro"/>
-  <!-- black_dount -->
+<robot name="kobuki" xmlns:xacro="http://ros.org/wiki/xacro">
+  <xacro:include filename="$(find chefbot_description)/urdf/common_properties.urdf.xacro"/>
+  <xacro:include filename="$(find chefbot_description)/urdf/chefbot_base_gazebo.urdf.xacro"/>
+  <!-- Kobuki -->
   <xacro:macro name="kobuki">
-    <!--link name="base_footprint"/-->
+    <link name="base_footprint"/>
     <!--
        Base link is set at the bottom of the base mould.
@@ -21,17 +21,17 @@
        to 0.352.
       -->
-    <!--joint name="base_joint" type="fixed">
+    <joint name="base_joint" type="fixed">
       <origin xyz="0 0 0.0102" rpy="0 0 0" />
       <parent link="base_footprint"/>
       <child link="base_link" />
-    </joint-->
+    </joint>
     <link name="base_link">
       <visual>
         <geometry>
           <!-- new mesh -->
-          <mesh filename="package://black_dount_description/meshes/base_plate.dae" />
+          <mesh filename="package://chefbot_description/meshes/base_plate.dae" />
         </geometry>
 <!--        <origin xyz="0.001 0 0.05199" rpy="0 0 ${M_PI/2}"/> -->
-	 <origin xyz="0.001 0 -0.034" rpy="0 0 ${M_PI/2}"/>
+	  <origin xyz="0.001 0 -0.034" rpy="0 0 ${M_PI/2}"/>
       </visual>
       <collision>
@@ -57,15 +57,14 @@
       </inertial>
     </link>
-<!--
     <joint name="wheel_left_joint" type="continuous">
       <parent link="base_link"/>
-      <child link="black_dount_wheel_left_link"/>
+      <child link="wheel_left_link"/>
       <origin xyz="0 ${0.28/2} 0.026" rpy="${-M_PI/2} 0 0"/>
       <axis xyz="0 0 1"/>
     </joint>
-    <link name="black_dount_wheel_left_link">
+    <link name="wheel_left_link">
       <visual>
         <geometry>
-          <mesh filename="package://black_dount_description/meshes/wheel.dae"/>
+          <mesh filename="package://chefbot_description/meshes/wheel.dae"/>
         </geometry>
         <origin xyz="0 0 0" rpy="0 0 0"/>
@@ -87,12 +86,12 @@
     <joint name="wheel_right_joint" type="continuous">
       <parent link="base_link"/>
-      <child link="black_dount_wheel_right_link"/>
+      <child link="wheel_right_link"/>
       <origin xyz="0.00 -${0.28/2} 0.026" rpy="${-M_PI/2} 0 0"/>
       <axis xyz="0 0 1"/>
     </joint>
-    <link name="black_dount_wheel_right_link">
+    <link name="wheel_right_link">
       <visual>
         <geometry>
-          <mesh filename="package://black_dount_description/meshes/wheel.dae"/>
+          <mesh filename="package://chefbot_description/meshes/wheel.dae"/>
         </geometry>
         <origin xyz="0 0 0" rpy="0 0 0"/>
@@ -112,123 +111,10 @@
       </inertial>
     </link>
--->
-	  <link name="left_axle_link">
-	    <inertial>
-	      <origin xyz="0 -0.035 0.021"/>
-	      <mass value="0.01" />
-	      <inertia ixx="0.001" ixy="0.0" ixz="0.0"
-	        iyy="0.001" iyz="0.0" izz="0.001" />
-	    </inertial>
-	    <visual>
-	      <origin xyz="0 -0.035 0.021" rpy="0 1.5707 1.5707" />
-	      <geometry>
-            <cylinder radius="0.0045" length = "0.02"/>
-	      </geometry>
-          <material name ="light_grey" />
-	    </visual>
-	    <collision>
-	      <origin xyz="0 -0.035 0.021" rpy="0 1.5707 1.5707" />
-	      <geometry>
-            <cylinder radius="0.00635" length = "0.00635"/>
-	      </geometry>
-	    </collision>
-	  </link>
-	  <joint name="left_axle_joint" type="fixed">
-	    <origin xyz="0 0.171475 0.0178" rpy="0 0 0"/>
-	    <parent link="base_link"/>
-	    <child link="left_axle_link"/>
-	    <axis xyz="0 1 0"/>
-	  </joint>
-	  <link name="right_axle_link">
-	    <inertial>
-	      <origin xyz="0 0.035 0.021"/>
-	      <mass value="0.01" />
-	      <inertia ixx="0.001" ixy="0.0" ixz="0.0"
-	        iyy="0.001" iyz="0.0" izz="0.001" />
-	    </inertial>
-	    <visual>
-	      <origin xyz="0 0.035 0.02" rpy="0 1.5707 1.5707" />
-	      <geometry>
-            <cylinder radius="0.0045" length = "0.002"/>
-	      </geometry>
-          <material name ="light_grey" />
-	    </visual>
-	    <collision>
-	      <origin xyz="0 0.035 0.02" rpy="0 1.5707 1.5707" />
-	      <geometry>
-            <cylinder radius="0.0045" length = "0.002"/>
-	      </geometry>
-	    </collision>
-	  </link>
-	  <joint name="right_axle_joint" type="fixed">
-	    <origin xyz="0 -0.171475 0.0178" rpy="0 0 0"/>
-	    <parent link="base_link"/>
-	    <child link="right_axle_link"/>
-	    <axis xyz="0 1 0"/>
-	  </joint>
-	  <link name="left_wheel_link">
-	    <inertial>
-	      <origin xyz="0 -0.035 0.021"/>
-	      <mass value="0.01" />
-	      <inertia ixx="0.001" ixy="0.0" ixz="0.0"
-	        iyy="0.001" iyz="0.0" izz="0.001" />
-	    </inertial>
-	    <visual>
-	      <origin xyz="0 -0.035 0.021" rpy="0 1.5707 1.5707" />
-	      <geometry>
-            <cylinder radius="0.045" length = "0.02"/>
-	      </geometry>
-          <material name ="black" />
-	    </visual>
-	    <collision>
-	      <origin xyz="0 -0.035 0.021" rpy="0 1.5707 1.5707" />
-	      <geometry>
-            <cylinder radius="0.0762" length = "0.03175"/>
-	      </geometry>
-	    </collision>
-	  </link>
-        <!-- Fixed because we never rotate it anyway, it is just for show -->
-        <!-- NOTE This may prevent gazebo from working with this model -->
-	  <joint name="left_wheel_joint" type="fixed">
-	    <origin xyz="0 0.01905 0" rpy="0 0 0"/>
-	    <parent link="left_axle_link"/>
-	    <child link="left_wheel_link"/>
-	    <axis xyz="0 1 0"/>
-	  </joint>
-	  <link name="right_wheel_link">
-	    <inertial>
-	      <origin xyz="0 0.035 0.021"/>
-	      <mass value="0.01" />
-	      <inertia ixx="0.001" ixy="0.0" ixz="0.0"
-	        iyy="0.001" iyz="0.0" izz="0.001" />
-	    </inertial>
-	    <visual>
-	      <origin xyz="0 0.035 0.021" rpy="0 1.5707 1.5707" />
-	      <geometry>
-            <cylinder radius="0.045" length = "0.02"/>
-	      </geometry>
-          <material name ="black" />
-	    </visual>
-	    <collision>
-	      <origin xyz="0 0.035 0.021" rpy="0 1.5707 1.5707" />
-	      <geometry>
-            <cylinder radius="0.045" length = "0.02"/>
-	      </geometry>
-	    </collision>
-	  </link>
-        <!-- Fixed because we never rotate it anyway, it is just for show -->
-        <!-- NOTE This may prevent gazebo from working with this model -->
-	  <joint name="right_wheel_joint" type="fixed">
-	    <origin xyz="0 -0.01905 0" rpy="0 0 0"/>
-	    <parent link="right_axle_link"/>
-	    <child link="right_wheel_link"/>
-	    <axis xyz="0 1 0"/>
-	  </joint>
     <joint name="caster_front_joint" type="fixed">
       <parent link="base_link"/>
-      <child link="black_dount_caster_front_link"/>
+      <child link="caster_front_link"/>
       <origin xyz="0.115 0.0 0.007" rpy="${-M_PI/2} 0 0"/>
     </joint>
-    <link name="black_dount_caster_front_link">
+    <link name="caster_front_link">
       <collision>
         <geometry>
@@ -245,10 +131,10 @@
       </inertial>
     </link>
-    <joint name="black_dount_caster_back_joint" type="fixed">
-      <parent link="base_link"/>
-      <child link="black_dount_caster_back_link"/>
+    <joint name="caster_back_joint" type="fixed">
+      <parent link="base_link"/>
+      <child link="caster_back_link"/>
       <origin xyz="-0.135 0.0 0.009" rpy="${-M_PI/2} 0 0"/>
     </joint>
-    <link name="black_dount_caster_back_link">
+    <link name="caster_back_link">
       <collision>
         <geometry>

File: chefbot_description/urdf/sensors/kinect.urdf.xacro (robot description, xacro)
@@ -1,6 +1,6 @@
 <?xml version="1.0"?>
 <robot name="sensor_kinect" xmlns:xacro="http://ros.org/wiki/xacro">
-  <xacro:include filename="$(find black_dount_description)/urdf/black_dount_gazebo.urdf.xacro"/>
-  <xacro:include filename="$(find black_dount_description)/urdf/black_dount_properties.urdf.xacro"/>
+  <xacro:include filename="$(find chefbot_description)/urdf/chefbot_gazebo.urdf.xacro"/>
+  <xacro:include filename="$(find chefbot_description)/urdf/chefbot_properties.urdf.xacro"/>
   <!-- Parameterised in part by the values in turtlebot_properties.urdf.xacro -->
   <xacro:macro name="sensor_kinect" params="parent">
