Commit message: Drive::OK

File: black_donut_description/urdf/robot.urdf.xacro (robot description, xacro)
@@ -2,3 +2,4 @@
 <robot xmlns:xacro="http://www.ros.org/wiki/xacro"  name="robot">
     <xacro:include filename="robot_core.xacro" />
+    <xacro:include filename="gazebo_control.xacro" />
 </robot>

File: black_donut_description/urdf/robot_core.xacro (robot description, xacro)
@@ -14,14 +14,14 @@
         <color rgba="0 0 0 1"/>
     </material>
+    <!-- BASE_FOOTPRINT LINK -->
+    <link name="base_footprint">
+    </link>
     <!-- BASE LINK -->
-    <link name="base_link">
-    </link>
-    <!-- CHASSIS LINK -->
-    <joint name="chassis_joint" type="fixed">
-        <parent link="base_link"/>
-        <child link="chassis"/>
+    <joint name="base_link_joint" type="fixed">
+        <parent link="base_footprint"/>
+        <child link="base_link"/>
         <origin xyz="0 0 0"/>
     </joint>
-    <link name="chassis">
+    <link name="base_link">
         <visual>
             <origin xyz="0 0 0.075"/>
@@ -89,5 +89,5 @@
     <!-- CASTER WHEEL LINK -->
     <joint name="caster_wheel_f_joint" type="fixed">
-        <parent link="chassis"/>
+        <parent link="base_link"/>
         <child link="caster_wheel_f"/>
         <origin xyz="0.1 0 0"/>
@@ -110,5 +110,5 @@
     </link>
     <joint name="caster_wheel_joint_b" type="fixed">
-        <parent link="chassis"/>
+        <parent link="base_link"/>
         <child link="caster_wheel_b"/>
         <origin xyz="-0.1 0 0"/>
@@ -130,3 +130,22 @@
         </xacro:inertial_sphere>
     </link>
+    <gazebo reference="base_link">
+        <material>Gazebo/Black</material>
+    </gazebo>
+    <gazebo reference="right_wheel">
+        <material>Gazebo/Orange</material>
+    </gazebo>
+    <gazebo reference="left_wheel">
+        <material>Gazebo/Orange</material>
+    </gazebo>
+    <gazebo reference="caster_wheel_f">
+        <material>Gazebo/Black</material>
+        <mu1 value="0.001"/>
+        <mu2 value="0.001"/>
+    </gazebo>
+    <gazebo reference="caster_wheel_b">
+        <material>Gazebo/Black</material>
+        <mu1 value="0.001"/>
+        <mu2 value="0.001"/>
+    </gazebo>
 </robot>
