Commit message: top_plate_added

File: black_donut_description/urdf/lidar.xacro (robot description, xacro)
@@ -9,5 +9,5 @@
         <visual>
             <geometry>
-                <cylinder radius="0.05" length="0.04"/>
+                <cylinder radius="0.05" length="0.06"/>
             </geometry>
             <material name="red"/>
@@ -15,8 +15,8 @@
         <collision>
             <geometry>
-                <cylinder radius="0.05" length="0.04"/>
+                <cylinder radius="0.05" length="0.06"/>
             </geometry>
         </collision>
-        <xacro:inertial_cylinder mass="0.1" length="0.04" radius="0.05">
+        <xacro:inertial_cylinder mass="0.1" length="0.06" radius="0.05">
             <origin xyz="0 0 0" rpy="0 0 0"/>
         </xacro:inertial_cylinder>

File: black_donut_description/urdf/robot_core.xacro (robot description, xacro)
@@ -39,4 +39,28 @@
         <xacro:inertial_box mass="0.5" x="0.3" y="0.3" z="0.15">
             <origin xyz="0 0 0.075" rpy="0 0 0"/>
+        </xacro:inertial_box>
+    </link>
+    <!-- TOP PLATE-->
+    <joint name="hat_joint" type="fixed">
+        <parent link="base_link"/>
+        <child link="hat_link"/>
+        <origin xyz="0 0 0"/>
+    </joint>
+    <link name="hat_link">
+        <visual>
+            <origin xyz="0 0 0.245"/>
+            <geometry>
+                <cylinder radius="0.2" length="0.01"/>
+            </geometry>1
+            <material name="black"/>
+        </visual>
+        <collision>
+            <origin xyz="0 0 0.245"/>
+            <geometry>
+                <box size="0.3 0.3 0.15"/>
+            </geometry>
+        </collision>
+        <xacro:inertial_box mass="0.1" x="0.1" y="0.1" z="0.1">
+            <origin xyz="0 0 0.245" rpy="0 0 0"/>
         </xacro:inertial_box>
     </link>
