Commit message: color and twist

File: black_donut_description/urdf/robot_core.xacro (robot description, xacro)
@@ -163,4 +163,9 @@
         <material>Gazebo/Orange</material>
     </gazebo>
+    <gazebo reference="hat_link">
+        <material>Gazebo/Black</material>
+        <mu1 value="0.001"/>
+        <mu2 value="0.001"/>
+    </gazebo>
     <gazebo reference="caster_wheel_f">
         <material>Gazebo/Black</material>
